File: Light-Gated-Noise-Box.sch (KiCad schematic (older format))
At the start: 10 parts, among them J1 Audio-Jack-2_Switch, U1 HEF4093B, U2 HEF4093B

Commit message: Final Draw
Parts:
- added R5: 1k, symbol R
- C1, C3: value C -> 100nF
- C2: value C -> 47nF
- R1, R2, R3, R4: value R_PHOTO -> 2M
Connections:
- net at R4.2, U2.11: now also R5.2; no longer J1.1
- new net: J1.1, R5.1
Other:
- note added: "I know this loop is weird\nBut it adds to the character :)"
- note removed: "Hoi"
- note removed: "I know this is weird\nBut it sounds awesome"
Changed lines of the file:
@@
 P 2300 3350
 F 0 "R1" H 2350 3400 50  0000 L CNN
-F 1 "R_PHOTO" H 2350 3350 50  0000 L TNN
+F 1 "2M" H 2350 3350 50  0000 L TNN
 F 2 "" V 2350 3100 50  0001 L CNN
 F 3 "" H 2300 3300 50  0001 C CNN
@@
 P 1850 3350
 F 0 "C1" H 1875 3450 50  0000 L CNN
-F 1 "C" H 1875 3250 50  0000 L CNN
+F 1 "100nF" H 1875 3250 50  0000 L CNN
 F 2 "" H 1888 3200 50  0001 C CNN
 F 3 "" H 1850 3350 50  0001 C CNN
@@
 $EndComp
 $Comp
-L GND #PWR01
+L GND #PWR3
 U 1 1 5A60E6F8
 P 1850 3850
-F 0 "#PWR01" H 1850 3600 50  0001 C CNN
+F 0 "#PWR3" H 1850 3600 50  0001 C CNN
 F 1 "GND" H 1850 3700 50  0000 C CNN
 F 2 "" H 1850 3850 50  0001 C CNN
@@
 	8600 2950 8600 3700
 Wire Wire Line
-	8600 3150 9900 3150
-Wire Wire Line
 	2300 3050 2300 3200
 Wire Wire Line
@@
 P 4100 3350
 F 0 "R2" H 4150 3400 50  0000 L CNN
-F 1 "R_PHOTO" H 4150 3350 50  0000 L TNN
+F 1 "2M" H 4150 3350 50  0000 L TNN
 F 2 "" V 4150 3100 50  0001 L CNN
 F 3 "" H 4100 3300 50  0001 C CNN
@@
 P 3650 3350
 F 0 "C2" H 3675 3450 50  0000 L CNN
-F 1 "C" H 3675 3250 50  0000 L CNN
+F 1 "47nF" H 3675 3250 50  0000 L CNN
 F 2 "" H 3688 3200 50  0001 C CNN
 F 3 "" H 3650 3350 50  0001 C CNN
@@
 $EndComp
 $Comp
-L GND #PWR02
+L GND #PWR4
 U 1 1 5A60E999
 P 3650 3850
-F 0 "#PWR02" H 3650 3600 50  0001 C CNN
+F 0 "#PWR4" H 3650 3600 50  0001 C CNN
 F 1 "GND" H 3650 3700 50  0000 C CNN
 F 2 "" H 3650 3850 50  0001 C CNN
@@
 P 5850 3350
 F 0 "R3" H 5900 3400 50  0000 L CNN
-F 1 "R_PHOTO" H 5900 3350 50  0000 L TNN
+F 1 "2M" H 5900 3350 50  0000 L TNN
 F 2 "" V 5900 3100 50  0001 L CNN
 F 3 "" H 5850 3300 50  0001 C CNN
@@
 P 7600 3350
 F 0 "R4" H 7650 3400 50  0000 L CNN
-F 1 "R_PHOTO" H 7650 3350 50  0000 L TNN
+F 1 "2M" H 7650 3350 50  0000 L TNN
 F 2 "" V 7650 3100 50  0001 L CNN
 F 3 "" H 7600 3300 50  0001 C CNN
@@
 P 7150 3350
 F 0 "C3" H 7175 3450 50  0000 L CNN
-F 1 "C" H 7175 3250 50  0000 L CNN
+F 1 "100nF" H 7175 3250 50  0000 L CNN
 F 2 "" H 7188 3200 50  0001 C CNN
 F 3 "" H 7150 3350 50  0001 C CNN
@@
 $EndComp
 $Comp
-L GND #PWR03
+L GND #PWR5
 U 1 1 5A60EBD0
 P 7150 3850
-F 0 "#PWR03" H 7150 3600 50  0001 C CNN
+F 0 "#PWR5" H 7150 3600 50  0001 C CNN
 F 1 "GND" H 7150 3700 50  0000 C CNN
 F 2 "" H 7150 3850 50  0001 C CNN
@@
 	5850 3050 6250 3050
 $Comp
-L GND #PWR04
+L GND #PWR2
 U 1 1 5A60EDB0
 P 1700 7200
-F 0 "#PWR04" H 1700 6950 50  0001 C CNN
+F 0 "#PWR2" H 1700 6950 50  0001 C CNN
 F 1 "GND" H 1700 7050 50  0000 C CNN
 F 2 "" H 1700 7200 50  0001 C CNN
@@
 	1700 7000 1700 7200
 $Comp
-L +9V #PWR05
+L +9V #PWR1
 U 1 1 5A60EE44
 P 1700 6200
-F 0 "#PWR05" H 1700 6050 50  0001 C CNN
+F 0 "#PWR1" H 1700 6050 50  0001 C CNN
 F 1 "+9V" H 1700 6340 50  0000 C CNN
 F 2 "" H 1700 6200 50  0001 C CNN
@@
 	1700 6200 1700 6400
 $Comp
-L PWR_FLAG #FLG06
+L PWR_FLAG #FLG1
 U 1 1 5A60EEFB
 P 1400 6200
-F 0 "#FLG06" H 1400 6275 50  0001 C CNN
+F 0 "#FLG1" H 1400 6275 50  0001 C CNN
 F 1 "PWR_FLAG" H 1400 6350 50  0000 C CNN
 F 2 "" H 1400 6200 50  0001 C CNN
@@
 	1400 6300 1700 6300
 Connection ~ 1700 6300
-Text Notes 5850 3950 0    60   ~ 0
-I know this is weird\nBut it sounds awesome
+Text Notes 5500 3950 0    60   ~ 0
+I know this loop is weird\nBut it adds to the character :)
 $Comp
 L HEF4093B U2
@@
 $EndComp
 $Comp
-L GND #PWR07
+L GND #PWR6
 U 1 1 5A60F55C
 P 10000 2650
-F 0 "#PWR07" H 10000 2400 50  0001 C CNN
+F 0 "#PWR6" H 10000 2400 50  0001 C CNN
 F 1 "GND" H 10000 2500 50  0000 C CNN
 F 2 "" H 10000 2650 50  0001 C CNN
@@
 	1400 7000 1700 7000
 Connection ~ 1400 6300
-Text Notes 4950 4900 0    60   ~ 0
-Hoi
+$Comp
+L R R5
+U 1 1 5A61FFBC
+P 9250 3150
+F 0 "R5" V 9330 3150 50  0000 C CNN
+F 1 "1k" V 9250 3150 50  0000 C CNN
+F 2 "" V 9180 3150 50  0001 C CNN
+F 3 "" H 9250 3150 50  0001 C CNN
+	1    9250 3150
+	0    1    1    0
+$EndComp
+Wire Wire Line
+	8600 3150 9100 3150
+Wire Wire Line
+	9400 3150 9900 3150
 $EndSCHEMATC

Commit message: Final draft
Parts:
- added D1, D2: LED, symbol LED
Connections:
- net +9V: now also D2.1 (K)
- net at R4.2, R5.2, U2.11: now also D1.2 (A)
- new net: D1.1 (K), D2.2 (A)
Changed lines of the file:
@@
 $EndComp
 $Comp
-L GND #PWR6
+L GND #PWR7
 U 1 1 5A60F55C
 P 10000 2650
-F 0 "#PWR6" H 10000 2400 50  0001 C CNN
+F 0 "#PWR7" H 10000 2400 50  0001 C CNN
 F 1 "GND" H 10000 2500 50  0000 C CNN
 F 2 "" H 10000 2650 50  0001 C CNN
@@
 Wire Wire Line
 	9400 3150 9900 3150
+$Comp
+L LED D1
+U 1 1 5A620316
+P 8950 3500
+F 0 "D1" H 8950 3600 50  0000 C CNN
+F 1 "LED" H 8950 3400 50  0000 C CNN
+F 2 "" H 8950 3500 50  0001 C CNN
+F 3 "" H 8950 3500 50  0001 C CNN
+	1    8950 3500
+	0    -1   -1   0
+$EndComp
+$Comp
+L LED D2
+U 1 1 5A62037E
+P 8950 3950
+F 0 "D2" H 8950 4050 50  0000 C CNN
+F 1 "LED" H 8950 3850 50  0000 C CNN
+F 2 "" H 8950 3950 50  0001 C CNN
+F 3 "" H 8950 3950 50  0001 C CNN
+	1    8950 3950
+	0    -1   -1   0
+$EndComp
+$Comp
+L GND #PWR6
+U 1 1 5A6203C9
+P 8950 4250
+F 0 "#PWR6" H 8950 4000 50  0001 C CNN
+F 1 "GND" H 8950 4100 50  0000 C CNN
+F 2 "" H 8950 4250 50  0001 C CNN
+F 3 "" H 8950 4250 50  0001 C CNN
+	1    8950 4250
+	1    0    0    -1
+$EndComp
+Wire Wire Line
+	8950 3350 8950 3150
+Connection ~ 8950 3150
+Wire Wire Line
+	8950 3650 8950 3800
+Wire Wire Line
+	8950 4100 8950 4250
 $EndSCHEMATC

Commit message: Final draft
Parts:
- R5: value 1k -> 220r
Connections:
- net +9V: now also R5.1; no longer D2.1 (K)
- net at D1.2 (A), R4.2, U2.11: now also J1.1; no longer R5.2
- new net: D2.1 (K), R5.2
Other:
- note added: "+"
- moved on the sheet: R5
Changed lines of the file:
@@
 L R R5
 U 1 1 5A61FFBC
-P 9250 3150
-F 0 "R5" V 9330 3150 50  0000 C CNN
-F 1 "1k" V 9250 3150 50  0000 C CNN
-F 2 "" V 9180 3150 50  0001 C CNN
-F 3 "" H 9250 3150 50  0001 C CNN
-	1    9250 3150
-	0    1    1    0
+P 8950 4400
+F 0 "R5" V 9030 4400 50  0000 C CNN
+F 1 "220r" V 8850 4400 50  0000 C CNN
+F 2 "" V 8880 4400 50  0001 C CNN
+F 3 "" H 8950 4400 50  0001 C CNN
+	1    8950 4400
+	-1   0    0    1
 $EndComp
 Wire Wire Line
-	8600 3150 9100 3150
-Wire Wire Line
-	9400 3150 9900 3150
+	8600 3150 9900 3150
 $Comp
 L LED D1
@@
 L GND #PWR6
 U 1 1 5A6203C9
-P 8950 4250
-F 0 "#PWR6" H 8950 4000 50  0001 C CNN
-F 1 "GND" H 8950 4100 50  0000 C CNN
-F 2 "" H 8950 4250 50  0001 C CNN
-F 3 "" H 8950 4250 50  0001 C CNN
-	1    8950 4250
+P 8950 4700
+F 0 "#PWR6" H 8950 4450 50  0001 C CNN
+F 1 "GND" H 8950 4550 50  0000 C CNN
+F 2 "" H 8950 4700 50  0001 C CNN
+F 3 "" H 8950 4700 50  0001 C CNN
+	1    8950 4700
 	1    0    0    -1
 $EndComp
@@
 Wire Wire Line
 	8950 4100 8950 4250
+Text Notes 2350 3200 0    60   ~ 0
++
+Text Notes 4150 3550 0    60   ~ 0
++
+Text Notes 5900 3550 0    60   ~ 0
++
+Text Notes 7650 3200 0    60   ~ 0
++
+Wire Wire Line
+	8950 4550 8950 4700
 $EndSCHEMATC
